File: CustomController/schematic/hexControllerV2/hexControllerV2.kicad_sch (KiCad schematic)
At the start: 48 parts, among them IC1 ESP32-S2-MINI-1-N4R2, IC2 IP5306, J1 USB_C_Receptacle_USB2.0_16P, J2 Battery, J3 Switch1, J4 Switch2, J5 Switch3, J6 Switch4, J7 Battery, SW1 RotaryEncoder_Switch, SW2 SW_DIP_x01, SW3 SW_DIP_x01, SW4 SW_DIP_x01, SW5 SW_DIP_x01, SW6 SW_DIP_x01, U2 AMS1117-3.3

Commit message: Reworking schematic
Other:
- moved on the sheet: C1, C10, C11, C12, C13, C14, C2, C3, C4, C5, C6, C8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
