Commit message: Add RViz configuration and update URDF properties for hexapod model

File: Hexapod/ros2/hexapod_ws/src/hexapod_description/urdf/hexapod.urdf.xacro (robot description, xacro)
@@ -2,4 +2,9 @@
 <robot xmlns:xacro="http://ros.org/wiki/xacro" name="hexapod">
   <!-- ================= CONSTANTS ================= -->
+  <xacro:property name="coxa_length" value="0.055"/>
+  <xacro:property name="femur_length" value="0.09"/>
+  <xacro:property name="tibia_length" value="0.15"/>
+  <xacro:property name="femur_radius" value="0.029"/>
+  <xacro:property name="tibia_radius" value="0.0225"/>
   <!-- ================= MATERIALS ================= -->
   <material name="black"><color rgba="0.1 0.1 0.1 1"/></material>
@@ -14,5 +19,5 @@
     <visual>
       <geometry>
-        <mesh filename="package://hexapod_description/meshes/body.dae" scale="0.01 0.01 0.01"/>
+        <mesh filename="package://hexapod_description/meshes/body.dae" scale="0.001 0.001 0.001"/>
       </geometry>
       <material name="black"/>
@@ -24,7 +29,7 @@
   <link name="${name}_coxa">
     <visual>
+      <origin xyz="${coxa_length/2} 0 0" rpy="0 0 0"/>
       <geometry>
-        <mesh filename="package://hexapod_description/meshes/coxa.dae"
-              scale="0.01 0.01 0.01"/>
+        <box size="${coxa_length} 0.048 0.06"/>
       </geometry>
       <material name="${colour}"/>
@@ -34,8 +39,8 @@
   <link name="${name}_femur">
     <visual>
-      <origin xyz="0.045 0 0" rpy="0 0 0"/>
+      <!-- Cylinder base aligned with joint -->
+      <origin xyz="${femur_length/2} 0 0" rpy="0 -1.5708 0"/>
       <geometry>
-        <mesh filename="package://hexapod_description/meshes/femur.dae"
-              scale="0.01 0.01 0.01"/>
+        <cylinder length="${femur_length}" radius="${femur_radius}"/>
       </geometry>
       <material name="${colour}"/>
@@ -45,8 +50,7 @@
   <link name="${name}_tibia">
     <visual>
-      <origin xyz="0.075175 0 0" rpy="0 0 0"/>
+      <origin xyz="${tibia_length/2} 0 0" rpy="0 -1.5708 0"/>
       <geometry>
-        <mesh filename="package://hexapod_description/meshes/tibia.dae"
-              scale="0.01 0.01 0.01"/>
+        <cylinder length="${tibia_length}" radius="${tibia_radius}"/>
       </geometry>
       <material name="${colour}"/>
@@ -57,5 +61,5 @@
     <parent link="base_link"/>
     <child link="${name}_coxa"/>
-    <origin xyz="${x_offset} ${y_offset} 0" rpy="0 0 ${yaw}"/>
+    <origin xyz="${x_offset} ${y_offset} 0.02" rpy="0 0 ${yaw}"/>
     <axis xyz="0 0 1"/>
     <limit lower="-1.57" upper="1.57" effort="1" velocity="1"/>
@@ -65,5 +69,5 @@
     <parent link="${name}_coxa"/>
     <child link="${name}_femur"/>
-    <origin xyz="0.0505 0 0" rpy="0 0 0"/>
+    <origin xyz="${coxa_length} 0 0" rpy="0 0 0"/>
     <axis xyz="0 1 0"/>
     <limit lower="-1.57" upper="1.57" effort="1" velocity="1"/>
@@ -73,5 +77,5 @@
     <parent link="${name}_femur"/>
     <child link="${name}_tibia"/>
-    <origin xyz="0.09 0 0" rpy="0 0 0"/>
+    <origin xyz="${femur_length} 0 0" rpy="0 1.5708 0"/>
     <axis xyz="0 1 0"/>
     <limit lower="-1.57" upper="1.57" effort="1" velocity="1"/>
@@ -82,5 +86,5 @@
   <xacro:leg name="leg1" x_offset="0.06733" y_offset="0.0846" yaw="0.5236" colour="red"/>
   <!-- Middle left -->
-  <xacro:leg name="leg2" x_offset="0.090" y_offset="0" yaw="1.57" colour="green"/>
+  <xacro:leg name="leg2" x_offset="0.090" y_offset="0" yaw="0" colour="green"/>
   <!-- Rear left -->
   <xacro:leg name="leg3" x_offset="-0.06733" y_offset="0.0846" yaw="2.36" colour="blue"/>
@@ -88,5 +92,5 @@
   <xacro:leg name="leg4" x_offset="0.06733" y_offset="-0.0846" yaw="-0.5236" colour="yellow"/>
   <!-- Middle right -->
-  <xacro:leg name="leg5" x_offset="-0.090" y_offset="0" yaw="-1.57" colour="cyan"/>
+  <xacro:leg name="leg5" x_offset="-0.090" y_offset="0" yaw="-3.14159" colour="cyan"/>
   <!-- Rear right -->
   <xacro:leg name="leg6" x_offset="-0.06733" y_offset="-0.0846" yaw="-2.36" colour="magenta"/>

Commit message: Update coxa dimensions in hexapod URDF for improved leg geometry

File: Hexapod/ros2/hexapod_ws/src/hexapod_description/urdf/hexapod.urdf.xacro (robot description, xacro)
@@ -5,4 +5,6 @@
   <xacro:property name="femur_length" value="0.09"/>
   <xacro:property name="tibia_length" value="0.15"/>
+  <xacro:property name="coxa_width" value="0.048"/>
+  <xacro:property name="coxa_height" value="0.06"/>
   <xacro:property name="femur_radius" value="0.029"/>
   <xacro:property name="tibia_radius" value="0.0225"/>
@@ -31,5 +33,5 @@
       <origin xyz="${coxa_length/2} 0 0" rpy="0 0 0"/>
       <geometry>
-        <box size="${coxa_length} 0.048 0.06"/>
+        <box size="${coxa_length} ${coxa_width} ${coxa_height}"/>
       </geometry>
       <material name="${colour}"/>

Commit message: Add collision geometry for legs and body in hexapod URDF

File: Hexapod/ros2/hexapod_ws/src/hexapod_description/urdf/hexapod.urdf.xacro (robot description, xacro)
@@ -9,4 +9,5 @@
   <xacro:property name="femur_radius" value="0.029"/>
   <xacro:property name="tibia_radius" value="0.0225"/>
+  <xacro:property name="cscale" value="0.95"/>
   <!-- ================= MATERIALS ================= -->
   <material name="black"><color rgba="0.1 0.1 0.1 1"/></material>
@@ -25,4 +26,9 @@
       <material name="black"/>
     </visual>
+    <collision>
+      <geometry>
+        <mesh filename="package://hexapod_description/meshes/body.dae" scale="0.001 0.001 0.001"/>
+      </geometry>
+    </collision>
   </link>
 <!-- ================= LEG LINKS ================= -->
@@ -37,4 +43,10 @@
       <material name="${colour}"/>
     </visual>
+    <collision>
+      <origin xyz="${coxa_length/2} 0 0" rpy="0 0 0"/>
+      <geometry>
+        <box size="${coxa_length*cscale} ${coxa_width*cscale} ${coxa_height*cscale}"/>
+      </geometry>
+    </collision>
   </link>
   <!-- FEMUR -->
@@ -48,4 +60,10 @@
       <material name="${colour}"/>
     </visual>
+    <collision>
+      <origin xyz="${femur_length/2} 0 0" rpy="0 -1.5708 0"/>
+      <geometry>
+        <cylinder length="${femur_length*cscale}" radius="${femur_radius*cscale}"/>
+      </geometry>
+    </collision>
   </link>
   <!-- TIBIA -->
@@ -58,4 +76,10 @@
       <material name="${colour}"/>
     </visual>
+    <collision>
+      <origin xyz="${tibia_length/2} 0 0" rpy="0 -1.5708 0"/>
+      <geometry>
+        <cylinder length="${tibia_length*cscale}" radius="${tibia_radius*cscale}"/>
+      </geometry>
+    </collision>
   </link>
   <!-- COXA JOINT -->

Commit message: Update URDF file for hexapod: replace gazebo-specific model with simplified box geometry and add inertial properties; remove obsolete gazebo.urdf.xacro file.

File: Hexapod/ros2/hexapod_ws/src/hexapod_description/urdf/hexapod.urdf.xacro (robot description, xacro)
@@ -22,5 +22,6 @@
     <visual>
       <geometry>
-        <mesh filename="package://hexapod_description/meshes/body.dae" scale="0.001 0.001 0.001"/>
+        <box size="0.18 0.17 0.05"/>
+        <!--<mesh filename="package://hexapod_description/meshes/body.dae" scale="0.01 0.01 0.01"/>-->
       </geometry>
       <material name="black"/>
@@ -28,7 +29,13 @@
     <collision>
       <geometry>
-        <mesh filename="package://hexapod_description/meshes/body.dae" scale="0.001 0.001 0.001"/>
+        <box size="0.18 0.17 0.05"/>
+        <!--<mesh filename="package://hexapod_description/meshes/body.dae" scale="0.01 0.01 0.01"/>-->
       </geometry>
     </collision>
+    <inertial>
+      <mass value="1.0"/>
+      <origin xyz="0 0 0"/>
+      <inertia ixx="0.1" ixy="0.0" ixz="0.0" iyy="0.1" iyz="0.0" izz="0.1"/>
+    </inertial>
   </link>
 <!-- ================= LEG LINKS ================= -->
@@ -49,4 +56,9 @@
       </geometry>
     </collision>
+    <inertial>
+      <mass value="0.1"/>
+      <origin xyz="${coxa_length/2} 0 0"/>
+      <inertia ixx="0.01" ixy="0.0" ixz="0.0" iyy="0.01" iyz="0.0" izz="0.01"/>
+    </inertial>
   </link>
   <!-- FEMUR -->
@@ -66,4 +78,9 @@
       </geometry>
     </collision>
+    <inertial>
+      <mass value="0.05"/>
+      <origin xyz="${femur_length/2} 0 0"/>
+      <inertia ixx="0.001" ixy="0.0" ixz="0.0" iyy="0.001" iyz="0.0" izz="0.001"/>
+    </inertial>
   </link>
   <!-- TIBIA -->
@@ -82,4 +99,9 @@
       </geometry>
     </collision>
+    <inertial>
+      <mass value="0.05"/>
+      <origin xyz="${tibia_length/2} 0 0"/>
+      <inertia ixx="0.001" ixy="0.0" ixz="0.0" iyy="0.001" iyz="0.0" izz="0.001"/>
+    </inertial>
   </link>
   <!-- COXA JOINT -->
@@ -87,5 +109,5 @@
     <parent link="base_link"/>
     <child link="${name}_coxa"/>
-    <origin xyz="${x_offset} ${y_offset} 0.02" rpy="0 0 ${yaw}"/>
+    <origin xyz="${x_offset} ${y_offset} 0" rpy="0 0 ${yaw}"/>
     <axis xyz="0 0 1"/>
     <limit lower="-1.57" upper="1.57" effort="1" velocity="1"/>

Commit message: Add ROS2 control and transmission definitions for hexapod joints in URDF

File: Hexapod/ros2/hexapod_ws/src/hexapod_description/urdf/hexapod.urdf.xacro (robot description, xacro)
@@ -129,4 +129,37 @@
     <limit lower="-1.57" upper="1.57" effort="1" velocity="1"/>
   </joint>
+  <!-- COXA TRANSMISSION -->
+  <transmission name="${name}_coxa_trans">
+    <type>transmission_interface/SimpleTransmission</type>
+    <joint name="${name}_coxa_joint">
+      <hardwareInterface>PositionJointInterface</hardwareInterface>
+    </joint>
+    <actuator name="${name}_coxa_motor">
+      <hardwareInterface>PositionJointInterface</hardwareInterface>
+      <mechanicalReduction>1</mechanicalReduction>
+    </actuator>
+  </transmission>
+  <!-- FEMUR TRANSMISSION -->
+  <transmission name="${name}_femur_trans">
+    <type>transmission_interface/SimpleTransmission</type>
+    <joint name="${name}_femur_joint">
+      <hardwareInterface>PositionJointInterface</hardwareInterface>
+    </joint>
+    <actuator name="${name}_femur_motor">
+      <hardwareInterface>PositionJointInterface</hardwareInterface>
+      <mechanicalReduction>1</mechanicalReduction>
+    </actuator>
+  </transmission>
+  <!-- TIBIA TRANSMISSION -->
+  <transmission name="${name}_tibia _trans">
+    <type>transmission_interface/SimpleTransmission</type>
+    <joint name="${name}_tibia_joint">
+      <hardwareInterface>PositionJointInterface</hardwareInterface>
+    </joint>
+    <actuator name="${name}_tibia_motor">
+      <hardwareInterface>PositionJointInterface</hardwareInterface>
+      <mechanicalReduction>1</mechanicalReduction>
+    </actuator>
+  </transmission>
 </xacro:macro>
   <!-- ================= LEGS ================= -->
@@ -143,3 +176,37 @@
   <!-- Rear right -->
   <xacro:leg name="leg6" x_offset="-0.06733" y_offset="0.0846" yaw="2.61799" colour="magenta"/>
+  <!-- ================= ROS2 CONTROL ================= -->
+  <xacro:macro name="ros2_control_joint" params="joint_name">
+    <joint name="${joint_name}">
+      <command_interface name="position"/>
+      <state_interface name="position"/>
+      <state_interface name="velocity"/>
+    </joint>
+  </xacro:macro>
+  <ros2_control name="HexapodHardware" type="system">
+    <hardware>
+      <plugin>gazebo_ros2_control/GazeboSystem</plugin>
+    </hardware>
+    <xacro:ros2_control_joint joint_name="leg1_coxa_joint"/>
+    <xacro:ros2_control_joint joint_name="leg1_femur_joint"/>
+    <xacro:ros2_control_joint joint_name="leg1_tibia_joint"/>
+    <xacro:ros2_control_joint joint_name="leg2_coxa_joint"/>
+    <xacro:ros2_control_joint joint_name="leg2_femur_joint"/>
+    <xacro:ros2_control_joint joint_name="leg2_tibia_joint"/>
+    <xacro:ros2_control_joint joint_name="leg3_coxa_joint"/>
+    <xacro:ros2_control_joint joint_name="leg3_femur_joint"/>
+    <xacro:ros2_control_joint joint_name="leg3_tibia_joint"/>
+    <xacro:ros2_control_joint joint_name="leg4_coxa_joint"/>
+    <xacro:ros2_control_joint joint_name="leg4_femur_joint"/>
+    <xacro:ros2_control_joint joint_name="leg4_tibia_joint"/>
+    <xacro:ros2_control_joint joint_name="leg5_coxa_joint"/>
+    <xacro:ros2_control_joint joint_name="leg5_femur_joint"/>
+    <xacro:ros2_control_joint joint_name="leg5_tibia_joint"/>
+    <xacro:ros2_control_joint joint_name="leg6_coxa_joint"/>
+    <xacro:ros2_control_joint joint_name="leg6_femur_joint"/>
+    <xacro:ros2_control_joint joint_name="leg6_tibia_joint"/>
+  </ros2_control>
+  <gazebo>
+    <plugin name="gazebo_ros2_control" filename="libgazebo_ros2_control.so"/>
+  </gazebo>
 </robot>
