Commit message: Added meshes to robot URDF

File: ros2/hexapod_ws/src/hexapod_description/urdf/hexapod.urdf.xacro (robot description, xacro)
@@ -1,13 +1,8 @@
-<?xml version="1.0"?>
 <robot xmlns:xacro="http://ros.org/wiki/xacro" name="hexapod">
   <!-- ================= CONSTANTS ================= -->
-  <xacro:property name="coxa_length" value="0.055"/>
-  <xacro:property name="femur_length" value="0.09"/>
+  <xacro:property name="coxa_length" value="0.0375"/>
+  <xacro:property name="femur_length" value="0.1"/>
   <xacro:property name="tibia_length" value="0.15"/>
-  <xacro:property name="coxa_width" value="0.048"/>
-  <xacro:property name="coxa_height" value="0.06"/>
-  <xacro:property name="femur_radius" value="0.029"/>
-  <xacro:property name="tibia_radius" value="0.0225"/>
-  <xacro:property name="cscale" value="0.95"/>
+  <xacro:property name="femur_z_offset" value="0.0106"/>
   <!-- ================= MATERIALS ================= -->
   <material name="black"><color rgba="0.1 0.1 0.1 1"/></material>
@@ -22,6 +17,5 @@
     <visual>
       <geometry>
-        <box size="0.18 0.17 0.05"/>
-        <!--<mesh filename="package://hexapod_description/meshes/body.dae" scale="0.01 0.01 0.01"/>-->
+        <mesh filename="package://hexapod_description/meshes/body.fbx" scale="0.01 0.01 0.01"/>
       </geometry>
       <material name="black"/>
@@ -29,6 +23,5 @@
     <collision>
       <geometry>
-        <box size="0.18 0.17 0.05"/>
-        <!--<mesh filename="package://hexapod_description/meshes/body.dae" scale="0.01 0.01 0.01"/>-->
+        <mesh filename="package://hexapod_description/meshes/body.fbx" scale="0.01 0.01 0.01"/>
       </geometry>
     </collision>
@@ -44,19 +37,19 @@
   <link name="${name}_coxa">
     <visual>
-      <origin xyz="${coxa_length/2} 0 0" rpy="0 0 0"/>
-      <geometry>
-        <box size="${coxa_length} ${coxa_width} ${coxa_height}"/>
+      <origin xyz="0 0 0" rpy="0 0 1.5708"/>
+      <geometry>
+        <mesh filename="package://hexapod_description/meshes/coxa.fbx" scale="0.01 0.01 0.01"/>
       </geometry>
       <material name="${colour}"/>
     </visual>
     <collision>
-      <origin xyz="${coxa_length/2} 0 0" rpy="0 0 0"/>
-      <geometry>
-        <box size="${coxa_length*cscale} ${coxa_width*cscale} ${coxa_height*cscale}"/>
+      <origin xyz="0 0 0" rpy="0 0 1.5708"/>
+      <geometry>
+        <mesh filename="package://hexapod_description/meshes/coxa.fbx" scale="0.01 0.01 0.01"/>
       </geometry>
     </collision>
     <inertial>
       <mass value="0.1"/>
-      <origin xyz="${coxa_length/2} 0 0"/>
+      <origin xyz="0 0 0"/>
       <inertia ixx="0.01" ixy="0.0" ixz="0.0" iyy="0.01" iyz="0.0" izz="0.01"/>
     </inertial>
@@ -65,20 +58,19 @@
   <link name="${name}_femur">
     <visual>
-      <!-- Cylinder base aligned with joint -->
-      <origin xyz="${femur_length/2} 0 0" rpy="0 -1.5708 0"/>
-      <geometry>
-        <cylinder length="${femur_length}" radius="${femur_radius}"/>
+      <origin xyz="0 0 0" rpy="0 0 1.5708"/>
+      <geometry>
+        <mesh filename="package://hexapod_description/meshes/femur.fbx" scale="0.01 0.01 0.01"/>
       </geometry>
       <material name="${colour}"/>
     </visual>
     <collision>
-      <origin xyz="${femur_length/2} 0 0" rpy="0 -1.5708 0"/>
-      <geometry>
-        <cylinder length="${femur_length*cscale}" radius="${femur_radius*cscale}"/>
+      <origin xyz="0 0 0" rpy="0 0 1.5708"/>
+      <geometry>
+        <mesh filename="package://hexapod_description/meshes/femur.fbx" scale="0.01 0.01 0.01"/>
       </geometry>
     </collision>
     <inertial>
       <mass value="0.05"/>
-      <origin xyz="${femur_length/2} 0 0"/>
+      <origin xyz="0 0 0"/>
       <inertia ixx="0.001" ixy="0.0" ixz="0.0" iyy="0.001" iyz="0.0" izz="0.001"/>
     </inertial>
@@ -87,19 +79,19 @@
   <link name="${name}_tibia">
     <visual>
-      <origin xyz="${tibia_length/2} 0 0" rpy="0 -1.5708 0"/>
-      <geometry>
-        <cylinder length="${tibia_length}" radius="${tibia_radius}"/>
+      <origin xyz="0 0 0" rpy="0 0 1.5708"/>
+      <geometry>
+        <mesh filename="package://hexapod_description/meshes/tibia.fbx" scale="0.01 0.01 0.01"/>
       </geometry>
       <material name="${colour}"/>
     </visual>
     <collision>
-      <origin xyz="${tibia_length/2} 0 0" rpy="0 -1.5708 0"/>
-      <geometry>
-        <cylinder length="${tibia_length*cscale}" radius="${tibia_radius*cscale}"/>
+      <origin xyz="0 0 0" rpy="0 0 1.5708"/>
+      <geometry>
+        <mesh filename="package://hexapod_description/meshes/tibia.fbx" scale="0.01 0.01 0.01"/>
       </geometry>
     </collision>
     <inertial>
       <mass value="0.05"/>
-      <origin xyz="${tibia_length/2} 0 0"/>
+      <origin xyz="0 0 0"/>
       <inertia ixx="0.001" ixy="0.0" ixz="0.0" iyy="0.001" iyz="0.0" izz="0.001"/>
     </inertial>
@@ -117,5 +109,5 @@
     <parent link="${name}_coxa"/>
     <child link="${name}_femur"/>
-    <origin xyz="${coxa_length} 0 0" rpy="0 0 0"/>
+    <origin xyz="${coxa_length} 0 ${femur_z_offset}" rpy="0 0 0"/>
     <axis xyz="0 1 0"/>
     <limit lower="-1.57" upper="1.57" effort="1" velocity="1"/>

Commit message: Converted meshes to .dae format and included foxglove bridge on robot side

File: ros2/hexapod_ws/src/hexapod_description/urdf/hexapod.urdf.xacro (robot description, xacro)
@@ -5,4 +5,6 @@
   <xacro:property name="tibia_length" value="0.15"/>
   <xacro:property name="femur_z_offset" value="0.0106"/>
+  <xacro:property name="mesh_up_correction_rpy" value="-1.5708 0 0"/>
+  <xacro:property name="mesh_up_correction_with_yaw_rpy" value="-1.5708 0 1.5708"/>
   <!-- ================= MATERIALS ================= -->
   <material name="black"><color rgba="0.1 0.1 0.1 1"/></material>
@@ -16,12 +18,14 @@
   <link name="base_link">
     <visual>
-      <geometry>
-        <mesh filename="package://hexapod_description/meshes/body.fbx" scale="0.01 0.01 0.01"/>
+      <origin xyz="0 0 0" rpy="${mesh_up_correction_rpy}"/>
+      <geometry>
+        <mesh filename="package://hexapod_description/meshes/body.dae" scale="0.01 0.01 0.01"/>
       </geometry>
       <material name="black"/>
     </visual>
     <collision>
-      <geometry>
-        <mesh filename="package://hexapod_description/meshes/body.fbx" scale="0.01 0.01 0.01"/>
+      <origin xyz="0 0 0" rpy="${mesh_up_correction_rpy}"/>
+      <geometry>
+        <mesh filename="package://hexapod_description/meshes/body.dae" scale="0.01 0.01 0.01"/>
       </geometry>
     </collision>
@@ -37,14 +41,14 @@
   <link name="${name}_coxa">
     <visual>
-      <origin xyz="0 0 0" rpy="0 0 1.5708"/>
-      <geometry>
-        <mesh filename="package://hexapod_description/meshes/coxa.fbx" scale="0.01 0.01 0.01"/>
+      <origin xyz="0 0 0" rpy="${mesh_up_correction_with_yaw_rpy}"/>
+      <geometry>
+        <mesh filename="package://hexapod_description/meshes/coxa.dae" scale="0.01 0.01 0.01"/>
       </geometry>
       <material name="${colour}"/>
     </visual>
     <collision>
-      <origin xyz="0 0 0" rpy="0 0 1.5708"/>
-      <geometry>
-        <mesh filename="package://hexapod_description/meshes/coxa.fbx" scale="0.01 0.01 0.01"/>
+      <origin xyz="0 0 0" rpy="${mesh_up_correction_with_yaw_rpy}"/>
+      <geometry>
+        <mesh filename="package://hexapod_description/meshes/coxa.dae" scale="0.01 0.01 0.01"/>
       </geometry>
     </collision>
@@ -58,14 +62,14 @@
   <link name="${name}_femur">
     <visual>
-      <origin xyz="0 0 0" rpy="0 0 1.5708"/>
-      <geometry>
-        <mesh filename="package://hexapod_description/meshes/femur.fbx" scale="0.01 0.01 0.01"/>
+      <origin xyz="0 0 0" rpy="${mesh_up_correction_with_yaw_rpy}"/>
+      <geometry>
+        <mesh filename="package://hexapod_description/meshes/femur.dae" scale="0.01 0.01 0.01"/>
       </geometry>
       <material name="${colour}"/>
     </visual>
     <collision>
-      <origin xyz="0 0 0" rpy="0 0 1.5708"/>
-      <geometry>
-        <mesh filename="package://hexapod_description/meshes/femur.fbx" scale="0.01 0.01 0.01"/>
+      <origin xyz="0 0 0" rpy="${mesh_up_correction_with_yaw_rpy}"/>
+      <geometry>
+        <mesh filename="package://hexapod_description/meshes/femur.dae" scale="0.01 0.01 0.01"/>
       </geometry>
     </collision>
@@ -79,14 +83,14 @@
   <link name="${name}_tibia">
     <visual>
-      <origin xyz="0 0 0" rpy="0 0 1.5708"/>
-      <geometry>
-        <mesh filename="package://hexapod_description/meshes/tibia.fbx" scale="0.01 0.01 0.01"/>
+      <origin xyz="0 0 0" rpy="${mesh_up_correction_with_yaw_rpy}"/>
+      <geometry>
+        <mesh filename="package://hexapod_description/meshes/tibia.dae" scale="0.01 0.01 0.01"/>
       </geometry>
       <material name="${colour}"/>
     </visual>
     <collision>
-      <origin xyz="0 0 0" rpy="0 0 1.5708"/>
-      <geometry>
-        <mesh filename="package://hexapod_description/meshes/tibia.fbx" scale="0.01 0.01 0.01"/>
+      <origin xyz="0 0 0" rpy="${mesh_up_correction_with_yaw_rpy}"/>
+      <geometry>
+        <mesh filename="package://hexapod_description/meshes/tibia.dae" scale="0.01 0.01 0.01"/>
       </geometry>
     </collision>
