Commit message: Enhance Hexapod control: add joint state relay, update URDF, and configure controllers

File: ros2/hexapod_ws/src/hexapod_description/urdf/hexapod_primitives.urdf.xacro (robot description, xacro)
@@ -2,8 +2,12 @@
   <xacro:arg name="controllers_file" default=""/>
   <!-- ================= CONSTANTS ================= -->
-  <xacro:property name="coxa_length" value="0.0375"/>
-  <xacro:property name="femur_length" value="0.1"/>
+  <xacro:property name="coxa_length" value="0.055"/>
+  <xacro:property name="femur_length" value="0.09"/>
   <xacro:property name="tibia_length" value="0.15"/>
-  <xacro:property name="femur_z_offset" value="0.0106"/>
+  <xacro:property name="coxa_width" value="0.048"/>
+  <xacro:property name="coxa_height" value="0.06"/>
+  <xacro:property name="femur_radius" value="0.029"/>
+  <xacro:property name="tibia_radius" value="0.0225"/>
+  <xacro:property name="cscale" value="0.95"/>
   <!-- ================= MATERIALS ================= -->
   <material name="black"><color rgba="0.1 0.1 0.1 1"/></material>
@@ -18,5 +22,5 @@
     <visual>
       <geometry>
-        <mesh filename="package://hexapod_description/meshes/body.dae" scale="1 1 1"/>
+        <box size="0.18 0.17 0.05"/>
       </geometry>
       <material name="black"/>
@@ -24,5 +28,5 @@
     <collision>
       <geometry>
-        <mesh filename="package://hexapod_description/meshes/body.dae" scale="1 1 1"/>
+        <box size="0.18 0.17 0.05"/>
       </geometry>
     </collision>
@@ -38,19 +42,19 @@
   <link name="${name}_coxa">
     <visual>
-      <origin xyz="0 0 0" rpy="0 0 1.5708"/>
-      <geometry>
-        <mesh filename="package://hexapod_description/meshes/coxa.dae" scale="1 1 1"/>
+      <origin xyz="${coxa_length/2} 0 0" rpy="0 0 0"/>
+      <geometry>
+        <box size="${coxa_length} ${coxa_width} ${coxa_height}"/>
       </geometry>
       <material name="${colour}"/>
     </visual>
     <collision>
-      <origin xyz="0 0 0" rpy="0 0 1.5708"/>
-      <geometry>
-        <mesh filename="package://hexapod_description/meshes/coxa.dae" scale="1 1 1"/>
+      <origin xyz="${coxa_length/2} 0 0" rpy="0 0 0"/>
+      <geometry>
+        <box size="${coxa_length*cscale} ${coxa_width*cscale} ${coxa_height*cscale}"/>
       </geometry>
     </collision>
     <inertial>
       <mass value="0.1"/>
-      <origin xyz="0 0 0"/>
+      <origin xyz="${coxa_length/2} 0 0"/>
       <inertia ixx="0.01" ixy="0.0" ixz="0.0" iyy="0.01" iyz="0.0" izz="0.01"/>
     </inertial>
@@ -59,19 +63,20 @@
   <link name="${name}_femur">
     <visual>
-      <origin xyz="0 0 0" rpy="0 0 1.5708"/>
-      <geometry>
-        <mesh filename="package://hexapod_description/meshes/femur.dae" scale="1 1 1"/>
+      <!-- Cylinder base aligned with joint -->
+      <origin xyz="${femur_length/2} 0 0" rpy="0 -1.5708 0"/>
+      <geometry>
+        <cylinder length="${femur_length}" radius="${femur_radius}"/>
       </geometry>
       <material name="${colour}"/>
     </visual>
     <collision>
-      <origin xyz="0 0 0" rpy="0 0 1.5708"/>
-      <geometry>
-        <mesh filename="package://hexapod_description/meshes/femur.dae" scale="1 1 1"/>
+      <origin xyz="${femur_length/2} 0 0" rpy="0 -1.5708 0"/>
+      <geometry>
+        <cylinder length="${femur_length*cscale}" radius="${femur_radius*cscale}"/>
       </geometry>
     </collision>
     <inertial>
       <mass value="0.05"/>
-      <origin xyz="0 0 0"/>
+      <origin xyz="${femur_length/2} 0 0"/>
       <inertia ixx="0.001" ixy="0.0" ixz="0.0" iyy="0.001" iyz="0.0" izz="0.001"/>
     </inertial>
@@ -80,19 +85,19 @@
   <link name="${name}_tibia">
     <visual>
-      <origin xyz="0 0 0" rpy="0 0 1.5708"/>
-      <geometry>
-        <mesh filename="package://hexapod_description/meshes/tibia.dae" scale="1 1 1"/>
+      <origin xyz="${tibia_length/2} 0 0" rpy="0 -1.5708 0"/>
+      <geometry>
+        <cylinder length="${tibia_length}" radius="${tibia_radius}"/>
       </geometry>
       <material name="${colour}"/>
     </visual>
     <collision>
-      <origin xyz="0 0 0" rpy="0 0 1.5708"/>
-      <geometry>
-        <mesh filename="package://hexapod_description/meshes/tibia.dae" scale="1 1 1"/>
+      <origin xyz="${tibia_length/2} 0 0" rpy="0 -1.5708 0"/>
+      <geometry>
+        <cylinder length="${tibia_length*cscale}" radius="${tibia_radius*cscale}"/>
       </geometry>
     </collision>
     <inertial>
       <mass value="0.05"/>
-      <origin xyz="0 0 0"/>
+      <origin xyz="${tibia_length/2} 0 0"/>
       <inertia ixx="0.001" ixy="0.0" ixz="0.0" iyy="0.001" iyz="0.0" izz="0.001"/>
     </inertial>
@@ -110,5 +115,5 @@
     <parent link="${name}_coxa"/>
     <child link="${name}_femur"/>
-    <origin xyz="${coxa_length} 0 ${femur_z_offset}" rpy="0 0 0"/>
+    <origin xyz="${coxa_length} 0 0" rpy="0 0 0"/>
     <axis xyz="0 1 0"/>
     <limit lower="-1.57" upper="1.57" effort="1" velocity="1"/>
