Commit message: Add sensors to hexapod URDF: camera, front depth camera, IMU, and lidar
Co-authored-by: Copilot <copilot@github.com>

File: ros2/hexapod_ws/src/hexapod_description/urdf/hexapod_primitives.urdf.xacro (robot description, xacro)
@@ -174,4 +174,178 @@
   <!-- Rear right -->
   <xacro:leg name="leg6" x_offset="-0.06733" y_offset="0.0846" yaw="2.61799" colour="magenta"/>
+  <!-- ================= SENSORS ================= -->
+  <link name="camera_link">
+    <visual>
+      <geometry><box size="0.02 0.05 0"/></geometry>
+      <material name="black"/>
+    </visual>
+    <collision>
+      <geometry><box size="0.02 0.05 0.02"/></geometry>
+    </collision>
+    <inertial>
+      <mass value="0.1"/>
+      <inertia ixx="0.001" ixy="0.0" ixz="0.0" iyy="0.001" iyz="0.0" izz="0.001"/>
+    </inertial>
+  </link>
+  <joint name="camera_joint" type="fixed">
+    <parent link="base_link"/>
+    <child link="camera_link"/>
+    <origin xyz="0.0 0.0846 0" rpy="0 0 1.5708"/>
+  </joint>
+  <gazebo reference="camera_link">
+  <sensor name="camera" type="camera">
+    <always_on>true</always_on>
+    <update_rate>30</update_rate>
+    <camera>
+      <horizontal_fov>1.047</horizontal_fov>  <!-- 60 degrees -->
+      <image>
+        <width>640</width>
+        <height>480</height>
+        <format>R8G8B8</format>
+      </image>
+      <clip>
+        <near>0.01</near>
+        <far>100</far>
+      </clip>
+    </camera>
+    <topic>/camera/image</topic>
+    <gz_frame_id>camera_link</gz_frame_id>
+  </sensor>
+</gazebo>
+<link name="front_depth_camera_link">
+  <visual>
+    <geometry><box size="0.03 0.03 0.02"/></geometry>
+    <material name="black"/>
+  </visual>
+  <collision>
+    <geometry><box size="0.03 0.03 0.02"/></geometry>
+  </collision>
+  <inertial>
+    <mass value="0.08"/>
+    <inertia ixx="0.0005" ixy="0.0" ixz="0.0" iyy="0.0005" iyz="0.0" izz="0.0005"/>
+  </inertial>
+</link>
+<joint name="front_depth_camera_joint" type="fixed">
+  <parent link="base_link"/>
+  <child link="front_depth_camera_link"/>
+  <origin xyz="0.0 0.0846 0.02" rpy="0 0 1.5708"/>
+</joint>
+<gazebo reference="front_depth_camera_link">
+  <sensor name="front_depth_camera" type="depth_camera">
+    <always_on>true</always_on>
+    <update_rate>30</update_rate>
+    <camera>
+      <horizontal_fov>1.2043</horizontal_fov>
+      <image>
+        <width>640</width>
+        <height>480</height>
+        <format>R8G8B8</format>
+      </image>
+      <clip>
+        <near>0.2</near>
+        <far>10.0</far>
+      </clip>
+    </camera>
+    <topic>/front_depth</topic>
+    <gz_frame_id>front_depth_camera_link</gz_frame_id>
+  </sensor>
+</gazebo>
+<link name="imu_link">
+  <visual>
+    <geometry><box size="0.015 0.015 0.005"/></geometry>
+    <material name="green"/>
+  </visual>
+  <collision>
+    <geometry><box size="0.015 0.015 0.005"/></geometry>
+  </collision>
+  <inertial>
+    <mass value="0.01"/>
+    <inertia ixx="1e-6" ixy="0.0" ixz="0.0" iyy="1e-6" iyz="0.0" izz="1e-6"/>
+  </inertial>
+</link>
+<joint name="imu_joint" type="fixed">
+  <parent link="base_link"/>
+  <child link="imu_link"/>
+  <origin xyz="0.0 0.0 0.03" rpy="0 0 0"/>
+</joint>
+<gazebo reference="imu_link">
+  <sensor name="imu_sensor" type="imu">
+    <always_on>true</always_on>
+    <update_rate>100</update_rate>
+    <topic>/imu</topic>
+    <gz_frame_id>imu_link</gz_frame_id>
+    <imu>
+      <angular_velocity>
+        <x><noise type="gaussian"><mean>0.0</mean><stddev>0.002</stddev></noise></x>
+        <y><noise type="gaussian"><mean>0.0</mean><stddev>0.002</stddev></noise></y>
+        <z><noise type="gaussian"><mean>0.0</mean><stddev>0.002</stddev></noise></z>
+      </angular_velocity>
+      <linear_acceleration>
+        <x><noise type="gaussian"><mean>0.0</mean><stddev>0.02</stddev></noise></x>
+        <y><noise type="gaussian"><mean>0.0</mean><stddev>0.02</stddev></noise></y>
+        <z><noise type="gaussian"><mean>0.0</mean><stddev>0.02</stddev></noise></z>
+      </linear_acceleration>
+    </imu>
+  </sensor>
+</gazebo>
+<gazebo reference="imu_link">
+  <sensor name="mag_sensor" type="magnetometer">
+    <always_on>true</always_on>
+    <update_rate>50</update_rate>
+    <topic>/imu/mag</topic>
+    <gz_frame_id>imu_link</gz_frame_id>
+  </sensor>
+</gazebo>
+<link name="lidar_link">
+  <visual>
+    <geometry><cylinder length="0.04" radius="0.025"/></geometry>
+    <material name="black"/>
+  </visual>
+  <collision>
+    <geometry><cylinder length="0.04" radius="0.025"/></geometry>
+  </collision>
+  <inertial>
+    <mass value="0.1"/>
+    <inertia ixx="0.001" ixy="0" ixz="0" iyy="0.001" iyz="0" izz="0.001"/>
+  </inertial>
+</link>
+<joint name="lidar_joint" type="fixed">
+  <parent link="base_link"/>
+  <child link="lidar_link"/>
+  <origin xyz="0 0 0.05" rpy="0 0 0"/>  <!-- top of body -->
+</joint>
+<gazebo reference="lidar_link">
+  <sensor name="lidar" type="gpu_lidar">
+    <always_on>true</always_on>
+    <update_rate>10</update_rate>
+    <lidar>
+      <scan>
+        <horizontal>
+          <samples>800</samples>
+          <resolution>1</resolution>
+          <min_angle>-3.14159</min_angle>
+          <max_angle>3.14159</max_angle>
+        </horizontal>
+        <vertical>
+          <samples>1</samples>        <!-- 1 = 2D lidar, increase for 3D -->
+          <min_angle>0</min_angle>
+          <max_angle>0</max_angle>
+        </vertical>
+      </scan>
+      <range>
+        <min>0.2</min>
+        <max>12.0</max>
+        <resolution>0.01</resolution>
+      </range>
+      <noise>
+        <type>gaussian</type>
+        <mean>0.0</mean>
+        <stddev>0.01</stddev>
+      </noise>
+    </lidar>
+    <topic>/lidar/scan</topic>
+    <gz_frame_id>lidar_link</gz_frame_id>
+  </sensor>
+</gazebo>
   <!-- ================= ROS2 CONTROL ================= -->
   <xacro:macro name="ros2_control_joint" params="joint_name">
